Commit message: einstein urdf has correct axes and joint limits just need to measure correct dimensions

File: einstein_description/urdf/einstein_robot.urdf (robot description, URDF)
Before this commit: robot einstein_robot, 5 links, 5 joints
Joints:
- joint base_joint: child neck_yaw -> neck_yaw_link
- joint gaze_joint: origin xyz=0.0539 0 0.05 -> xyz=0.05 0 -0.1 rpy=0 1.57 0
- joint neck_pitch: axis 0 0 1 -> 0 1 0; origin xyz=0 0 0 rpy=0 0 0  -> xyz=0.1 0 0 rpy=-1.57 0 0
- joint neck_roll: axis 0 0 1 -> 0 1 0; limit lower=-2 upper=2.0 effort=30 velocity=0.78 -> lower=-0.8 upper=1.2 effort=30 velocity=0.78; origin xyz=0 0 0 rpy=0 0 0  -> xyz=0.1 0 0 rpy=1.57 0 0
- joint neck_yaw: axis 0 0 1 -> 1 0 0; origin xyz=0 0 0 rpy=0 0 0  -> xyz=0.1 0 0 rpy=0 -1.57 0
